Commit message: Added some robots
Signed-off-by: Michał <michal.pelka@robotec.ai>

File: URDFTest/02_IMPORTING_VALID_SIMPLE_URDF/data/chain.urdf (robot description, URDF)
Before this commit: robot urdf_test, 4 links, 3 joints
Links:
- link suzanne_link: geometry collision mesh filename=suzanne.stl; visual mesh filename=suzanne.stl

Commit message: Apply suggestions from code review
Co-authored-by: Jan Hanca <134940295+jhanca-robotecai@users.noreply.github.com>

File: URDFTest/02_IMPORTING_VALID_SIMPLE_URDF/data/chain.urdf (robot description, URDF)
Before this commit: robot urdf_test, 4 links, 3 joints
Links:
- link suzanne_link: geometry collision mesh filename=suzanne.stl; visual mesh filename=suzanne.dae
